File: Coin/Coin.kicad_pcb (KiCad board)
At the start: 2 copper layers, 20 x 20 mm, 9 parts, among them J1 Conn_02x03_Odd_Even, U1 MPU-6050

Commit message: Updated silkscreen
Parts:
- added G***: LOGO, Coin:hackzone, B.Cu at (71.8, 113.8)
Other:
- board text added: "TOKEN"
- board text removed: "VOUCH"
